File: led-strip-shift-register.kicad_pcb (KiCad board)
At the start: 4 copper layers, 65 x 56 mm, 18 parts, among them J3 40HAT, J6 CONN_02X02, J9 CONN_01X02, Q1 DMG2305UX, Q2 DMMT5401, U2 CAT24C32

Commit message: mostly done hopefully
Parts:
- removed R11, R7, R9: DNP, Resistor_SMD:R_0603_1608Metric_Pad0.84x1.00mm_HandSolder
- removed R29: 10K, Resistor_SMD:R_0603_1608Metric_Pad0.84x1.00mm_HandSolder
- removed R6, R8: 3.9K, Resistor_SMD:R_0603_1608Metric_Pad0.84x1.00mm_HandSolder
- added C1: 1u, Capacitor_SMD:C_0603_1608Metric, F.Cu at (122.9, 76.4)
- added C2: 1u, Capacitor_SMD:C_0603_1608Metric, F.Cu at (99.6, 78.2)
- added C3: 1u, Capacitor_SMD:C_0603_1608Metric, F.Cu at (96.0, 81.5)
- added C4: 1u, Capacitor_SMD:C_0603_1608Metric, F.Cu at (112.0, 83.0)
- added G***: LOGO, footprints:peragato, B.Cu at (111.9, 74.8)
- added J1: LED_0, Connector_PinSocket_2.54mm:PinSocket_1x04_P2.54mm_Vertical, F.Cu at (83.8, 99.1)
- added J10: LED_7, Connector_PinSocket_2.54mm:PinSocket_1x04_P2.54mm_Vertical, F.Cu at (106.2, 91.9)
- added J11: LED_8, Connector_PinSocket_2.54mm:PinSocket_1x04_P2.54mm_Vertical, F.Cu at (113.8, 105.9)
- added J12: LED_9, Connector_PinSocket_2.54mm:PinSocket_1x04_P2.54mm_Vertical, F.Cu at (113.8, 91.9)
- added J13: LED_A, Connector_PinSocket_2.54mm:PinSocket_1x04_P2.54mm_Vertical, F.Cu at (121.4, 105.9)
- added J14: LED_B, Connector_PinSocket_2.54mm:PinSocket_1x04_P2.54mm_Vertical, F.Cu at (121.4, 91.9)
- added J15: LED_C, Connector_PinSocket_2.54mm:PinSocket_1x04_P2.54mm_Vertical, F.Cu at (129.8, 99.1)
- added J16: LED_D, Connector_PinSocket_2.54mm:PinSocket_1x04_P2.54mm_Vertical, F.Cu at (129.8, 85.1)
- added J17: LED_E, Connector_PinSocket_2.54mm:PinSocket_1x04_P2.54mm_Vertical, F.Cu at (137.2, 99.1)
- added J18: LED_F, Connector_PinSocket_2.54mm:PinSocket_1x04_P2.54mm_Vertical, F.Cu at (137.2, 85.1)
- added J2: LED_1, Connector_PinSocket_2.54mm:PinSocket_1x04_P2.54mm_Vertical, F.Cu at (83.8, 85.1)
- added J4: LED_2, Connector_PinSocket_2.54mm:PinSocket_1x04_P2.54mm_Vertical, F.Cu at (91.2, 99.1)
- added J5: LED_3, Connector_PinSocket_2.54mm:PinSocket_1x04_P2.54mm_Vertical, F.Cu at (91.2, 85.1)
- added J7: LED_4, Connector_PinSocket_2.54mm:PinSocket_1x04_P2.54mm_Vertical, F.Cu at (98.6, 105.9)
- added J8: LED_5, Connector_PinSocket_2.54mm:PinSocket_1x04_P2.54mm_Vertical, F.Cu at (98.6, 91.9)
- added MK1: ICS-43434, footprints:I2S-MIC_DIP-6, F.Cu at (135.1, 74.4)
- added U1: SN74HC163, Package_SO:SOIC-16_3.9x9.9mm_P1.27mm, F.Cu at (116.1, 73.2)
- added U3: 74HCT595D,118, footprints:SOIC127P600X175-16N, F.Cu at (103.1, 83.3)
- added U4: 74HCT595D,118, footprints:SOIC127P600X175-16N, F.Cu at (118.4, 83.1)
- J6: value CONN_02X02 -> POWER; footprint Connector_PinHeader_2.54mm:PinHeader_2x02_P2.54mm_Vertical -> TerminalBlock:TerminalBlock_bornier-2_P5.08mm
- J9: value CONN_01X02 -> LED_6; footprint Connector_PinHeader_2.54mm:PinHeader_1x02_P2.54mm_Vertical -> Connector_PinSocket_2.54mm:PinSocket_1x04_P2.54mm_Vertical
- U2: value CAT24C32 -> 74HCT244; footprint Package_SOIC:SOIC-8_3.9x4.9mm_P1.27mm -> Package_SO:TSSOP-20_4.4x6.5mm_P0.65mm
- moved J9 32.7 mm to (106.2, 105.9), turned to 0 degrees
- moved U2 17.8 mm to (102.6, 73.4)
- moved J6 11.6 mm to (82.3, 73.3), turned to 270 degrees
- moved R23 10.7 mm to (95.8, 70.7), turned to 0 degrees
- moved R24 10.6 mm to (95.8, 68.4), turned to 0 degrees
- moved Q2 5.59 mm to (92.3, 69.5), turned to 90 degrees
- moved Q1 1.20 mm to (88.7, 70.0), turned to 270 degrees
Connections:
- J3 pad 1: /P3V3_HAT -> +3V3
- J3 pad 10: (no net) -> Net-(J3-Pad10)
- J3 pad 11: (no net) -> Net-(J3-Pad11)
- J3 pad 12: (no net) -> /I2S_CLK
- J3 pad 13: (no net) -> /~CNT_LOAD
- J3 pad 15: (no net) -> /~RST
- J3 pad 16: (no net) -> Net-(J3-Pad16)
- J3 pad 17: (no net) -> +3V3
- J3 pad 18: (no net) -> Net-(J3-Pad18)
- J3 pad 19: (no net) -> /DAT
- J3 pad 2: /P5V_HAT -> +5V
- J3 pad 21: (no net) -> Net-(J3-Pad21)
- J3 pad 22: (no net) -> Net-(J3-Pad22)
- J3 pad 23: (no net) -> /CLK
- J3 pad 24: (no net) -> /CNT_ENA
- J3 pad 26: (no net) -> Net-(J3-Pad26)
- J3 pad 27: /ID_SD_EEPROM -> Net-(J3-Pad27)
- J3 pad 28: /ID_SC_EEPROM -> Net-(J3-Pad28)
- J3 pad 29: (no net) -> /CNT_P3
- J3 pad 3: (no net) -> Net-(J3-Pad3)
- J3 pad 31: (no net) -> /CNT_P2
- J3 pad 32: (no net) -> Net-(J3-Pad32)
- J3 pad 33: (no net) -> /CNT_P1
- J3 pad 35: (no net) -> /CNT_P0
- J3 pad 36: (no net) -> Net-(J3-Pad36)
- J3 pad 37: (no net) -> /I2S_WS
- J3 pad 38: (no net) -> /I2S_IN
- J3 pad 4: /P5V_HAT -> +5V
- J3 pad 40: (no net) -> Net-(J3-Pad40)
- J3 pad 5: (no net) -> Net-(J3-Pad5)
- J3 pad 7: (no net) -> Net-(J3-Pad7)
- J3 pad 8: (no net) -> Net-(J3-Pad8)
- J6 pad 1: /P3V3 -> GND
- J6 pad 2: /P3V3_HAT -> +5VP
- J9 pad 1: GND -> +5VP
- J9 pad 2: Net-(J9-Pad2) -> /L6
- Q1 pad 2: /P5V_HAT -> +5V
- Q1 pad 3: /P5V -> +5VP
- Q2 pad 5: /P5V_HAT -> +5V
- Q2 pad 6: /P5V -> +5VP
- U2 pad 2: GND -> /CLK_DIV
- U2 pad 3: GND -> /LCLK
- U2 pad 4: GND -> /CLK_DIV
- U2 pad 5: /ID_SD_EEPROM -> /LCLK
- U2 pad 6: /ID_SC_EEPROM -> /CLK_DIV
- U2 pad 7: Net-(J9-Pad2) -> /LCLK
- U2 pad 8: /P3V3 -> /CLK_DIV
Routing:
- net /LCLK: track 0.00 -> 360.8 mm, vias 0 -> 4
- net +5VP: track 0.00 -> 179.6 mm
- net +5V: track 0.00 -> 56.4 mm, vias 0 -> 2
- net +3V3: track 0.00 -> 53.9 mm, vias 0 -> 1
- net /~RST: track 0.00 -> 53.4 mm, vias 0 -> 2
- net /I2S_CLK: track 0.00 -> 42.3 mm
- net /CLK: track 0.00 -> 36.5 mm, vias 0 -> 3
- net /LE: track 0.00 -> 32.5 mm, vias 0 -> 1
- net /CLK_DIV: track 0.00 -> 32.3 mm
- net /P3V3: track 31.3 -> 0.00 mm
- net /L8: track 0.00 -> 30.1 mm
- net /L0: track 0.00 -> 28.1 mm
- net /LA: track 0.00 -> 25.4 mm
- net /L4: track 0.00 -> 24.2 mm
- net /L6: track 0.00 -> 23.8 mm
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- added copper zone on F.Cu, net +5V
- added copper zone on B.Cu, net GND
- removed copper zone on B.Cu, net /P3V3_HAT
- removed copper zone on F.Cu, net /P5V
- removed copper zone on B.Cu, net /P5V_HAT
- removed copper zone on F.Cu, net /P5V_HAT
- removed copper zone on In2.Cu, net GND
Other:
- copper layers 4 -> 2
- board text added: "peragwin@gmail.com 02-07-2021 github.com/peragwin/led-strip-shift-register"
- board text removed: "If you want to use an SMT 40-pin header, please move the top edge up by 0.5mm and locate the header in the same location as the current TH part."
- board text removed: "This is a HAT compatible PCB starting design based on the official Raspberry Pi specs at: https://github.com/raspberrypi/hats/blob/master/designguide.md Currently the camera slot and display cutout are not here. See the schematic for the details on the EEPROM and power setup. This board does have the correct components for powering the Pi via the HAT. If you need the Pi to provide 5V or 3.3V, ple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"

Commit message: revisions for components
Parts:
- added R1: 10k, Resistor_SMD:R_0603_1608Metric_Pad0.98x0.95mm_HandSolder, F.Cu at (96.4, 77.3)
- C1, C2, C3, C4: footprint Capacitor_SMD:C_0603_1608Metric -> Capacitor_SMD:C_0603_1608Metric_Pad1.08x0.95mm_HandSolder
- U1: value SN74HC163 -> SN74LV163A
- renumbered J12 to J10, J13 to J11, J14 to J12, J15 to J13, J16 to J14, J17 to J15, J18 to J16, J3 to J17, J6 to J18, J4 to J3, J5 to J4, J7 to J5, J8 to J6, J9 to J7, J10 to J8, J11 to J9
Connections:
- J17 pad 11: Net-(J3-Pad11) -> /~LCLK_OE
- U2 pad 1: GND -> /~LCLK_OE
- U2 pad 19: GND -> /~LCLK_OE
Routing:
- net /~LCLK_OE: track 0.00 -> 20.4 mm, vias 0 -> 1
- net GND: track 8.87 -> 3.40 mm, vias 8 -> 9
- net /LCLK: track 360.8 -> 364.4 mm
- net +5V: track 56.4 -> 59.5 mm

Commit message: tweaks before submission
Parts:
- added R2: 10k, Resistor_SMD:R_0603_1608Metric_Pad0.98x0.95mm_HandSolder, F.Cu at (125.1, 73.4)
- renumbered R23 to R3, R24 to R4
