File: led-strip-shift-register.sch (KiCad schematic (older format))
At the start: 15 parts, among them J3 40HAT, J6 CONN_02X02, Q1 DMG2305UX, Q2 DMMT5401

Commit message: mostly done hopefully
Parts:
- removed J6: CONN_02X02, Connector_PinHeader_2.54mm:PinHeader_2x02_P2.54mm_Vertical, symbol Connector_Generic:Conn_02x02_Odd_Even
- removed R7, R9: DNP, Resistor_SMD:R_0603_1608Metric_Pad0.84x1.00mm_HandSolder, symbol Device:R
- added C1, C2, C3, C4: 1u, Capacitor_SMD:C_0603_1608Metric, symbol Device:C
- added J1: LED_0, Connector_PinSocket_2.54mm:PinSocket_1x04_P2.54mm_Vertical, symbol Connector_Generic:Conn_01x04
- added J10: LED_7, Connector_PinSocket_2.54mm:PinSocket_1x04_P2.54mm_Vertical, symbol Connector_Generic:Conn_01x04
- added J11: LED_8, Connector_PinSocket_2.54mm:PinSocket_1x04_P2.54mm_Vertical, symbol Connector_Generic:Conn_01x04
- added J12: LED_9, Connector_PinSocket_2.54mm:PinSocket_1x04_P2.54mm_Vertical, symbol Connector_Generic:Conn_01x04
- added J13: LED_A, Connector_PinSocket_2.54mm:PinSocket_1x04_P2.54mm_Vertical, symbol Connector_Generic:Conn_01x04
- added J14: LED_B, Connector_PinSocket_2.54mm:PinSocket_1x04_P2.54mm_Vertical, symbol Connector_Generic:Conn_01x04
- added J15: LED_C, Connector_PinSocket_2.54mm:PinSocket_1x04_P2.54mm_Vertical, symbol Connector_Generic:Conn_01x04
- added J16: LED_D, Connector_PinSocket_2.54mm:PinSocket_1x04_P2.54mm_Vertical, symbol Connector_Generic:Conn_01x04
- added J17: LED_E, Connector_PinSocket_2.54mm:PinSocket_1x04_P2.54mm_Vertical, symbol Connector_Generic:Conn_01x04
- added J18: LED_F, Connector_PinSocket_2.54mm:PinSocket_1x04_P2.54mm_Vertical, symbol Connector_Generic:Conn_01x04
- added J2: LED_1, Connector_PinSocket_2.54mm:PinSocket_1x04_P2.54mm_Vertical, symbol Connector_Generic:Conn_01x04
- added J4: LED_2, Connector_PinSocket_2.54mm:PinSocket_1x04_P2.54mm_Vertical, symbol Connector_Generic:Conn_01x04
- added J5: LED_3, Connector_PinSocket_2.54mm:PinSocket_1x04_P2.54mm_Vertical, symbol Connector_Generic:Conn_01x04
- added J6: POWER, TerminalBlock:TerminalBlock_bornier-2_P5.08mm, symbol Connector_Generic:Conn_01x02
- added J7: LED_4, Connector_PinSocket_2.54mm:PinSocket_1x04_P2.54mm_Vertical, symbol Connector_Generic:Conn_01x04
- added J8: LED_5, Connector_PinSocket_2.54mm:PinSocket_1x04_P2.54mm_Vertical, symbol Connector_Generic:Conn_01x04
- added J9: LED_6, Connector_PinSocket_2.54mm:PinSocket_1x04_P2.54mm_Vertical, symbol Connector_Generic:Conn_01x04
- added MK1: ICS-43434, footprints:I2S-MIC_DIP-6, symbol ICS-43434_DIP-6:ICS-43434
- added U2: 74HCT244, Package_SO:TSSOP-20_4.4x6.5mm_P0.65mm, symbol 74xx:74HCT244
- J3: symbol raspberrypi_hat:OX40HAT -> led-strip-shift-register-rescue:OX40HAT-raspberrypi_hat
- Q1: symbol raspberrypi_hat:DMG2305UX -> led-strip-shift-register-rescue:DMG2305UX-raspberrypi_hat
- Q2: symbol raspberrypi_hat:DMMT5401 -> led-strip-shift-register-rescue:DMMT5401-raspberrypi_hat
- U1: renamed from U?; Field4 C338758 -> (none); LCSC (none) -> C338758
- U3, U4: renamed from U?; footprint SOIC127P600X175-16N -> footprints:SOIC127P600X175-16N; symbol 74HCT595D_118:74HCT595D,118 -> led-strip-shift-register-rescue:74HCT595D,118-74HCT595D_118; LCSC (none) -> C282339
Connections:
- net P3V3_HAT is gone; now on net +3V3: J3.1 (P3V3)
- net P5V_HAT is gone; now on net +5V: J3.2 (P5V), J3.4 (P5V), Q1.2 (S), Q2.5 (E)
- net VCC is gone; now on net +3V3: U1.16 (VCC)
- net +5V: now also C2.1, C3.1, C4.1, U2.20 (VCC); no longer Q1.3 (D), Q2.6 (E), U3.10 (~MR), U4.10 (~MR)
- net CLK: now also J3.23 (BCM11)
- net CLK_DIV: now also U2.11 (2A3), U2.13 (2A2), U2.15 (2A1), U2.17 (2A0), U2.2 (1A0), U2.4 (1A1), U2.6 (1A2), U2.8 (1A3)
- net GND: now also C1.2, C2.2, C3.2, C4.2, J1.4 (Pin_4), J10.4 (Pin_4), J11.4 (Pin_4), J12.4 (Pin_4), J13.4 (Pin_4), J14.4 (Pin_4), J15.4 (Pin_4), J16.4 (Pin_4), J17.4 (Pin_4), J18.4 (Pin_4), J2.4 (Pin_4), J4.4 (Pin_4), J5.4 (Pin_4), J6.1 (Pin_1), J7.4 (Pin_4), J8.4 (Pin_4), J9.4 (Pin_4), MK1.3 (GND), MK1.6 (LR), U2.1 (1OE), U2.10 (GND), U2.19 (2OE)
- net I2S_CLK: now reaches J3.12 (BCM18)
- net I2S_CLK: now also MK1.4 (SCK)
- net ~CNT_LOAD: now reaches J3.13 (BCM27)
- net ~CNT_LOAD: now also U1.9 (~Pe)
- net ~RST: now reaches J3.15 (BCM22)
- net ~RST: now also U1.1 (~MR), U3.10 (~MR), U4.10 (~MR)
- net +3V3: now reaches J3.17 (P3V3)
- net +3V3: now also U1.7 (ENP), C1.1, MK1.2 (VDD)
- net DAT: now reaches J3.19 (BCM10)
- net DAT: now also U3.14 (DS)
- net CNT_ENA: now reaches J3.24 (BCM8)
- net CNT_ENA: now also U1.10 (ENT)
- net CNT_P3: now reaches J3.29 (BCM5)
- net CNT_P3: now also U1.6 (P3)
- net CNT_P2: now reaches J3.31 (BCM6)
- net CNT_P2: now also U1.5 (P2)
- net CNT_P1: now reaches J3.33 (BCM13)
- net CNT_P1: now also U1.4 (P1)
- net CNT_P0: now reaches J3.35 (BCM19)
- net CNT_P0: now also U1.3 (P0)
- net I2S_WS: now reaches J3.37 (BCM26)
- net I2S_WS: now also MK1.5 (WS)
- net I2S_IN: now reaches J3.38 (BCM20)
- net I2S_IN: now also MK1.1 (SD)
- net L1: now reaches U3.1 (Q1)
- net L1: now also J2.2 (Pin_2)
- net L0: now reaches U3.15 (Q0)
- net L0: now also J1.2 (Pin_2)
- net L2: now reaches U3.2 (Q2)
- net L2: now also J4.2 (Pin_2)
- net L3: now reaches U3.3 (Q3)
- net L3: now also J5.2 (Pin_2)
- net L4: now reaches U3.4 (Q4)
- net L4: now also J7.2 (Pin_2)
- net L5: now reaches U3.5 (Q5)
- net L5: now also J8.2 (Pin_2)
- net L6: now reaches U3.6 (Q6)
- net L6: now also J9.2 (Pin_2)
- net L7: now reaches U3.7 (Q7)
- net L7: now also J10.2 (Pin_2)
- net L9: now reaches U4.1 (Q1)
- net L9: now also J12.2 (Pin_2)
- net L8: now reaches U4.15 (Q0)
- net L8: now also J11.2 (Pin_2)
- net LA: now reaches U4.2 (Q2)
- net LA: now also J13.2 (Pin_2)
- net LB: now reaches U4.3 (Q3)
- net LB: now also J14.2 (Pin_2)
- net LC: now reaches U4.4 (Q4)
- net LC: now also J15.2 (Pin_2)
- net LD: now reaches U4.5 (Q5)
- net LD: now also J16.2 (Pin_2)
- net LE: now reaches U4.6 (Q6)
- net LE: now also J17.2 (Pin_2)
- net LF: now reaches U4.7 (Q7)
- net LF: now also J18.2 (Pin_2)
- net ID_SC_EEPROM: no longer names the net of J3.28 (BCM1)
- net ID_SD_EEPROM: no longer names the net of J3.27 (BCM0)
- new net +5VP: J1.1 (Pin_1), J10.1 (Pin_1), J11.1 (Pin_1), J12.1 (Pin_1), J13.1 (Pin_1), J14.1 (Pin_1), J15.1 (Pin_1), J16.1 (Pin_1), J17.1 (Pin_1), J18.1 (Pin_1), J2.1 (Pin_1), J4.1 (Pin_1), J5.1 (Pin_1), J6.2 (Pin_2), J7.1 (Pin_1), J8.1 (Pin_1), J9.1 (Pin_1), Q1.3 (D), Q2.6 (E)
- new net LCLK: J1.3 (Pin_3), J10.3 (Pin_3), J11.3 (Pin_3), J12.3 (Pin_3), J13.3 (Pin_3), J14.3 (Pin_3), J15.3 (Pin_3), J16.3 (Pin_3), J17.3 (Pin_3), J18.3 (Pin_3), J2.3 (Pin_3), J4.3 (Pin_3), J5.3 (Pin_3), J7.3 (Pin_3), J8.3 (Pin_3), J9.3 (Pin_3), U2.12 (1Y3), U2.14 (1Y2), U2.16 (1Y1), U2.18 (1Y0), U2.3 (2Y0), U2.5 (2Y1), U2.7 (2Y2), U2.9 (2Y3)
Other:
- note removed: "FLEXIBLE POWER SELECTION"
- note removed: "HAT spec indicates to NEVER\npower the 3.3V pins on the Raspberry Pi \nfrom the HAT header. Only connect the 3.3V\npower from the Pi if the HAT does not have\n3.3V on board.\n\nIF you are designing a board that could\neither be powered by the Pi or from the HAT\nthe jumpers here can be used.\n\nIn most cases, either design the HAT \nto provide the 5V to the Pi and use the\nprotection circuit abov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"
- moved on the sheet: U1, U3, U4

Commit message: revisions for components
Parts:
- added R1: 10k, Resistor_SMD:R_0603_1608Metric_Pad0.98x0.95mm_HandSolder, symbol Device:R
- C1, C2, C3, C4: footprint Capacitor_SMD:C_0603_1608Metric -> Capacitor_SMD:C_0603_1608Metric_Pad1.08x0.95mm_HandSolder
- J17: renamed from J3; symbol led-strip-shift-register-rescue:OX40HAT-raspberrypi_hat -> led-strip-shift-register-rescue:OX40HAT-raspberrypi_hat-led-strip-shift-register-rescue
- MK1: symbol ICS-43434_DIP-6:ICS-43434 -> led-strip-shift-register-rescue:ICS-43434-ICS-43434_DIP-6
- Q1: symbol led-strip-shift-register-rescue:DMG2305UX-raspberrypi_hat -> led-strip-shift-register-rescue:DMG2305UX-raspberrypi_hat-led-strip-shift-register-rescue
- Q2: symbol led-strip-shift-register-rescue:DMMT5401-raspberrypi_hat -> led-strip-shift-register-rescue:DMMT5401-raspberrypi_hat-led-strip-shift-register-rescue
- U1: value SN74HC163 -> SN74LV163A; LCSC C338758 -> (none)
- U3, U4: symbol led-strip-shift-register-rescue:74HCT595D,118-74HCT595D_118 -> led-strip-shift-register-rescue:74HCT595D,118-74HCT595D_118-led-strip-shift-register-rescue
- renumbered J12 to J10, J13 to J11, J14 to J12, J15 to J13, J16 to J14, J17 to J15, J18 to J16, J6 to J18, J4 to J3, J5 to J4, J7 to J5, J8 to J6, J9 to J7, J10 to J8, J11 to J9
Connections:
- net +5V: now also R1.1
- net GND: no longer U2.1 (1OE), U2.19 (2OE)
- net ~LCLK_OE: now reaches J17.11 (BCM17)
- net ~LCLK_OE: now also U2.1 (1OE), U2.19 (2OE), R1.2
Changed lines of the file:
@@
 $EndComp
 $Comp
-L led-strip-shift-register-rescue:OX40HAT-raspberrypi_hat J3
+L led-strip-shift-register-rescue:OX40HAT-raspberrypi_hat-led-strip-shift-register-rescue J17
 U 1 1 58DFC771
 P 2600 2250
-F 0 "J3" H 2950 2350 50  0000 C CNN
+F 0 "J17" H 2950 2350 50  0000 C CNN
 F 1 "40HAT" H 2300 2350 50  0000 C CNN
 F 2 "Connector_PinSocket_2.54mm:PinSocket_2x20_P2.54mm_Vertical" H 2600 2450 50  0001 C CNN
@@
 This is the recommended 5V rail protection for \na HAT with power going to the Pi.\nSee https://github.com/raspberrypi/hats/blob/master/designguide.md#back-powering-the-pi-via-the-j8-gpio-header
 $Comp
-L led-strip-shift-register-rescue:DMG2305UX-raspberrypi_hat Q1
+L led-strip-shift-register-rescue:DMG2305UX-raspberrypi_hat-led-strip-shift-register-rescue Q1
 U 1 1 58E14EB1
 P 2550 7500
@@
 $EndComp
 $Comp
-L led-strip-shift-register-rescue:DMMT5401-raspberrypi_hat Q2
+L led-strip-shift-register-rescue:DMMT5401-raspberrypi_hat-led-strip-shift-register-rescue Q2
 U 1 1 58E1538B
 P 2250 8100
@@
 $EndComp
 $Comp
-L led-strip-shift-register-rescue:DMMT5401-raspberrypi_hat Q2
+L led-strip-shift-register-rescue:DMMT5401-raspberrypi_hat-led-strip-shift-register-rescue Q2
 U 2 1 58E153D6
 P 2850 8100
@@
 	2150 7500 2300 7500
 $Comp
-L led-strip-shift-register-rescue:74HCT595D,118-74HCT595D_118 U3
+L led-strip-shift-register-rescue:74HCT595D,118-74HCT595D_118-led-strip-shift-register-rescue U3
 U 1 1 6021579D
 P 11000 2250
@@
 $EndComp
 $Comp
-L led-strip-shift-register-rescue:74HCT595D,118-74HCT595D_118 U4
+L led-strip-shift-register-rescue:74HCT595D,118-74HCT595D_118-led-strip-shift-register-rescue U4
 U 1 1 60215F22
 P 11000 4400
@@
 P 7050 4050
 F 0 "U1" H 7050 4816 50  0000 C CNN
-F 1 "SN74HC163" H 7050 4725 50  0000 C CNN
+F 1 "SN74LV163A" H 7050 4725 50  0000 C CNN
 F 2 "Package_SO:SOIC-16_3.9x9.9mm_P1.27mm" H 7050 4050 50  0001 C CNN
-F 3 "https://datasheet.lcsc.com/szlcsc/1811271815_Texas-Instruments-TI-SN74HC163DR_C338758.pdf" H 7050 4050 50  0001 C CNN
-F 4 "C338758" H 7050 4050 50  0001 C CNN "LCSC"
+F 3 "https://www.ti.com/lit/ds/symlink/sn74lv163a.pdf?HQS=dis-dk-null-digikeymode-dsf-pf-null-wwe&ts=1612728661129" H 7050 4050 50  0001 C CNN
 	1    7050 4050
 	1    0    0    -1
@@
 Wire Wire Line
 	8100 7000 8100 7100
-Wire Wire Line
-	8100 7400 8600 7400
-Connection ~ 8100 7100
-Wire Wire Line
-	8100 7100 8100 7400
 Connection ~ 8600 7400
 Text Label 11700 1850 0    50   ~ 0
@@
 	1450 2250 800  2250
 $Comp
-L Connector_Generic:Conn_01x04 J18
+L Connector_Generic:Conn_01x04 J16
 U 1 1 602BB40A
 P 13650 8900
-F 0 "J18" H 13730 8892 50  0000 L CNN
+F 0 "J16" H 13730 8892 50  0000 L CNN
 F 1 "LED_F" H 13730 8801 50  0000 L CNN
 F 2 "Connector_PinSocket_2.54mm:PinSocket_1x04_P2.54mm_Vertical" H 13650 8900 50  0001 C CNN
@@
 	13250 2100 13450 2100
 $Comp
-L Connector_Generic:Conn_01x04 J4
+L Connector_Generic:Conn_01x04 J3
 U 1 1 602EBA5F
 P 13650 2400
-F 0 "J4" H 13730 2392 50  0000 L CNN
+F 0 "J3" H 13730 2392 50  0000 L CNN
 F 1 "LED_2" H 13730 2301 50  0000 L CNN
 F 2 "Connector_PinSocket_2.54mm:PinSocket_1x04_P2.54mm_Vertical" H 13650 2400 50  0001 C CNN
@@
 	13250 2600 13450 2600
 $Comp
-L Connector_Generic:Conn_01x04 J5
+L Connector_Generic:Conn_01x04 J4
 U 1 1 602F163A
 P 13650 2900
-F 0 "J5" H 13730 2892 50  0000 L CNN
+F 0 "J4" H 13730 2892 50  0000 L CNN
 F 1 "LED_3" H 13730 2801 50  0000 L CNN
 F 2 "Connector_PinSocket_2.54mm:PinSocket_1x04_P2.54mm_Vertical" H 13650 2900 50  0001 C CNN
@@
 	13250 3100 13450 3100
 $Comp
-L Connector_Generic:Conn_01x04 J7
+L Connector_Generic:Conn_01x04 J5
 U 1 1 602F7943
 P 13650 3400
-F 0 "J7" H 13730 3392 50  0000 L CNN
+F 0 "J5" H 13730 3392 50  0000 L CNN
 F 1 "LED_4" H 13730 3301 50  0000 L CNN
 F 2 "Connector_PinSocket_2.54mm:PinSocket_1x04_P2.54mm_Vertical" H 13650 3400 50  0001 C CNN
@@
 	13250 3600 13450 3600
 $Comp
-L Connector_Generic:Conn_01x04 J8
+L Connector_Generic:Conn_01x04 J6
 U 1 1 602FE239
 P 13650 3900
-F 0 "J8" H 13730 3892 50  0000 L CNN
+F 0 "J6" H 13730 3892 50  0000 L CNN
 F 1 "LED_5" H 13730 3801 50  0000 L CNN
 F 2 "Connector_PinSocket_2.54mm:PinSocket_1x04_P2.54mm_Vertical" H 13650 3900 50  0001 C CNN
@@
 	13250 4100 13450 4100
 $Comp
-L Connector_Generic:Conn_01x04 J9
+L Connector_Generic:Conn_01x04 J7
 U 1 1 60305695
 P 13650 4400
-F 0 "J9" H 13730 4392 50  0000 L CNN
+F 0 "J7" H 13730 4392 50  0000 L CNN
 F 1 "LED_6" H 13730 4301 50  0000 L CNN
 F 2 "Connector_PinSocket_2.54mm:PinSocket_1x04_P2.54mm_Vertical" H 13650 4400 50  0001 C CNN
@@
 	13250 4600 13450 4600
 $Comp
-L Connector_Generic:Conn_01x04 J10
+L Connector_Generic:Conn_01x04 J8
 U 1 1 6030CC70
 P 13650 4900
-F 0 "J10" H 13730 4892 50  0000 L CNN
+F 0 "J8" H 13730 4892 50  0000 L CNN
 F 1 "LED_7" H 13730 4801 50  0000 L CNN
 F 2 "Connector_PinSocket_2.54mm:PinSocket_1x04_P2.54mm_Vertical" H 13650 4900 50  0001 C CNN
@@
 	13250 5000 13450 5000
 $Comp
-L Connector_Generic:Conn_01x04 J11
+L Connector_Generic:Conn_01x04 J9
 U 1 1 6031449E
 P 13650 5400
-F 0 "J11" H 13730 5392 50  0000 L CNN
+F 0 "J9" H 13730 5392 50  0000 L CNN
 F 1 "LED_8" H 13730 5301 50  0000 L CNN
 F 2 "Connector_PinSocket_2.54mm:PinSocket_1x04_P2.54mm_Vertical" H 13650 5400 50  0001 C CNN
@@
 	13250 5600 13450 5600
 $Comp
-L Connector_Generic:Conn_01x04 J12
+L Connector_Generic:Conn_01x04 J10
 U 1 1 6031BD3A
 P 13650 5900
-F 0 "J12" H 13730 5892 50  0000 L CNN
+F 0 "J10" H 13730 5892 50  0000 L CNN
 F 1 "LED_9" H 13730 5801 50  0000 L CNN
 F 2 "Connector_PinSocket_2.54mm:PinSocket_1x04_P2.54mm_Vertical" H 13650 5900 50  0001 C CNN
@@
 	13250 5100 13450 5100
 $Comp
-L Connector_Generic:Conn_01x04 J13
+L Connector_Generic:Conn_01x04 J11
 U 1 1 6038C9BB
 P 13650 6400
-F 0 "J13" H 13730 6392 50  0000 L CNN
+F 0 "J11" H 13730 6392 50  0000 L CNN
 F 1 "LED_A" H 13730 6301 50  0000 L CNN
 F 2 "Connector_PinSocket_2.54mm:PinSocket_1x04_P2.54mm_Vertical" H 13650 6400 50  0001 C CNN
@@
 	13250 6600 13450 6600
 $Comp
-L Connector_Generic:Conn_01x04 J14
+L Connector_Generic:Conn_01x04 J12
 U 1 1 6039E708
 P 13650 6900
-F 0 "J14" H 13730 6892 50  0000 L CNN
+F 0 "J12" H 13730 6892 50  0000 L CNN
 F 1 "LED_B" H 13730 6801 50  0000 L CNN
 F 2 "Connector_PinSocket_2.54mm:PinSocket_1x04_P2.54mm_Vertical" H 13650 6900 50  0001 C CNN
@@
 	13250 7100 13450 7100
 $Comp
-L Connector_Generic:Conn_01x04 J15
+L Connector_Generic:Conn_01x04 J13
 U 1 1 603A7A03
 P 13650 7400
-F 0 "J15" H 13730 7392 50  0000 L CNN
+F 0 "J13" H 13730 7392 50  0000 L CNN
 F 1 "LED_C" H 13730 7301 50  0000 L CNN
 F 2 "Connector_PinSocket_2.54mm:PinSocket_1x04_P2.54mm_Vertical" H 13650 7400 50  0001 C CNN
@@
 	13250 7600 13450 7600
 $Comp
-L Connector_Generic:Conn_01x04 J16
+L Connector_Generic:Conn_01x04 J14
 U 1 1 603B14BD
 P 13650 7900
-F 0 "J16" H 13730 7892 50  0000 L CNN
+F 0 "J14" H 13730 7892 50  0000 L CNN
 F 1 "LED_D" H 13730 7801 50  0000 L CNN
 F 2 "Connector_PinSocket_2.54mm:PinSocket_1x04_P2.54mm_Vertical" H 13650 7900 50  0001 C CNN
@@
 	13250 8100 13450 8100
 $Comp
-L Connector_Generic:Conn_01x04 J17
+L Connector_Generic:Conn_01x04 J15
 U 1 1 603BB4D6
 P 13650 8400
-F 0 "J17" H 13730 8392 50  0000 L CNN
+F 0 "J15" H 13730 8392 50  0000 L CNN
 F 1 "LED_E" H 13730 8301 50  0000 L CNN
 F 2 "Connector_PinSocket_2.54mm:PinSocket_1x04_P2.54mm_Vertical" H 13650 8400 50  0001 C CNN
@@
 	4400 2750 3200 2750
 $Comp
-L ICS-43434_DIP-6:ICS-43434 MK1
+L led-strip-shift-register-rescue:ICS-43434-ICS-43434_DIP-6 MK1
 U 1 1 6046383A
 P 7900 9200
@@
 F 0 "C1" H 8865 9196 50  0000 L CNN
 F 1 "1u" H 8865 9105 50  0000 L CNN
-F 2 "Capacitor_SMD:C_0603_1608Metric" H 8788 9000 50  0001 C CNN
+F 2 "Capacitor_SMD:C_0603_1608Metric_Pad1.08x0.95mm_HandSolder" H 8788 9000 50  0001 C CNN
 F 3 "~" H 8750 9150 50  0001 C CNN
 	1    8750 9150
@@
 F 0 "C3" H 9915 4246 50  0000 L CNN
 F 1 "1u" H 9915 4155 50  0000 L CNN
-F 2 "Capacitor_SMD:C_0603_1608Metric" H 9838 4050 50  0001 C CNN
+F 2 "Capacitor_SMD:C_0603_1608Metric_Pad1.08x0.95mm_HandSolder" H 9838 4050 50  0001 C CNN
 F 3 "~" H 9800 4200 50  0001 C CNN
 	1    9800 4200
@@
 F 0 "C2" H 9915 1846 50  0000 L CNN
 F 1 "1u" H 9915 1755 50  0000 L CNN
-F 2 "Capacitor_SMD:C_0603_1608Metric" H 9838 1650 50  0001 C CNN
+F 2 "Capacitor_SMD:C_0603_1608Metric_Pad1.08x0.95mm_HandSolder" H 9838 1650 50  0001 C CNN
 F 3 "~" H 9800 1800 50  0001 C CNN
 	1    9800 1800
@@
 F 0 "C4" H 9965 6596 50  0000 L CNN
 F 1 "1u" H 9965 6505 50  0000 L CNN
-F 2 "Capacitor_SMD:C_0603_1608Metric" H 9888 6400 50  0001 C CNN
+F 2 "Capacitor_SMD:C_0603_1608Metric_Pad1.08x0.95mm_HandSolder" H 9888 6400 50  0001 C CNN
 F 3 "~" H 9850 6550 50  0001 C CNN
 	1    9850 6550
@@
 5VP
 $Comp
-L Connector_Generic:Conn_01x02 J6
+L Connector_Generic:Conn_01x02 J18
 U 1 1 606ACDCA
 P 4750 9000
-F 0 "J6" H 4668 8675 50  0000 C CNN
+F 0 "J18" H 4668 8675 50  0000 C CNN
 F 1 "POWER" H 4850 8750 50  0000 C CNN
 F 2 "TerminalBlock:TerminalBlock_bornier-2_P5.08mm" H 4750 9000 50  0001 C CNN
@@
 	1    0    0    -1
 $EndComp
+Text Label 800  2750 0    50   ~ 0
+~LCLK_OE
+Wire Wire Line
+	800  2750 2000 2750
+Text Label 7650 7000 0    50   ~ 0
+~LCLK_OE
+Connection ~ 8100 7000
+$Comp
+L Device:R R1
+U 1 1 6026D4B4
+P 7350 6850
+F 0 "R1" H 7420 6896 50  0000 L CNN
+F 1 "10k" H 7420 6805 50  0000 L CNN
+F 2 "Resistor_SMD:R_0603_1608Metric_Pad0.98x0.95mm_HandSolder" V 7280 6850 50  0001 C CNN
+F 3 "~" H 7350 6850 50  0001 C CNN
+	1    7350 6850
+	1    0    0    -1
+$EndComp
+Wire Wire Line
+	7350 7000 8100 7000
+$Comp
+L power:+5V #PWR015
+U 1 1 6027B36B
+P 7350 6700
+F 0 "#PWR015" H 7350 6550 50  0001 C CNN
+F 1 "+5V" H 7450 6750 50  0000 C CNN
+F 2 "" H 7350 6700 50  0001 C CNN
+F 3 "" H 7350 6700 50  0001 C CNN
+	1    7350 6700
+	1    0    0    -1
+$EndComp

Commit message: tweaks before submission
Parts:
- added R2: 10k, Resistor_SMD:R_0603_1608Metric_Pad0.98x0.95mm_HandSolder, symbol Device:R
- renumbered R23 to R3, R24 to R4
Connections:
- net GND: now also R2.2
- net ~RST: now also R2.1
Changed lines of the file:
@@
 $EndComp
 $Comp
-L Device:R R23
+L Device:R R3
 U 1 1 58E15896
 P 2150 8700
-F 0 "R23" V 2230 8700 50  0000 C CNN
+F 0 "R3" V 2230 8700 50  0000 C CNN
 F 1 "10K" V 2150 8700 50  0000 C CNN
 F 2 "Resistor_SMD:R_0603_1608Metric_Pad0.84x1.00mm_HandSolder" V 2080 8700 50  0001 C CNN
@@
 $EndComp
 $Comp
-L Device:R R24
+L Device:R R4
 U 1 1 58E158A1
 P 2950 8700
-F 0 "R24" V 3030 8700 50  0000 C CNN
+F 0 "R4" V 3030 8700 50  0000 C CNN
 F 1 "47K" V 2950 8700 50  0000 C CNN
 F 2 "Resistor_SMD:R_0603_1608Metric_Pad0.84x1.00mm_HandSolder" V 2880 8700 50  0001 C CNN
@@
 F 1 "74HCT595D,118" H 11000 2929 50  0000 C CNN
 F 2 "footprints:SOIC127P600X175-16N" H 11000 2250 50  0001 L BNN
-F 3 "" H 11000 2250 50  0001 L BNN
+F 3 "https://rocelec.widen.net/view/pdf/umsr6rbkih/PHGL-S-A0000283114-1.pdf?t.download=true&u=5oefqw" H 11000 2250 50  0001 L BNN
 F 4 "1826641" H 11000 2250 50  0001 L BNN "OC_FARNELL"
 F 5 "78R7401" H 11000 2250 50  0001 L BNN "OC_NEWARK"
@@
 Text Label 9750 2250 0    50   ~ 0
 ~RST
-Wire Wire Line
-	9750 2250 10300 2250
 Text Label 800  3150 0    50   ~ 0
 DAT
@@
 	1    0    0    -1
 $EndComp
+$Comp
+L Device:R R2
+U 1 1 6022CDBD
+P 9350 2750
+F 0 "R2" H 9420 2796 50  0000 L CNN
+F 1 "10k" H 9420 2705 50  0000 L CNN
+F 2 "Resistor_SMD:R_0603_1608Metric_Pad0.98x0.95mm_HandSolder" V 9280 2750 50  0001 C CNN
+F 3 "~" H 9350 2750 50  0001 C CNN
+	1    9350 2750
+	1    0    0    -1
+$EndComp
+Wire Wire Line
+	10200 2950 9350 2950
+Wire Wire Line
+	9350 2950 9350 2900
+Wire Wire Line
+	9350 2600 9350 2250
+Wire Wire Line
+	9350 2250 10300 2250
 $EndSCHEMATC
